File: electronics/view_base/_autosave-view_base.kicad_sch (KiCad schematic)
At the start: 107 parts, among them J1 BLDC, J2 USB_C_Receptacle_USB2.0, J3 LCD, J4 A, J5 B, Q1 MMBT4403, Q2 UMH3N, U1 MT6701-CT, U10 ESP32-S3-WROOM-1-N8R8, U4 CP2102N-A02-GQFN28, U4 HX711, U5 TMC6300, U7 SN74LV1T34DBV, U8 VEML7700, U9 TS1117BCW33_RPG

Commit message: Updated to esp32s3, cp2102, re-routed
Parts:
- U9: footprint Modified:SOT-223-3_TabPin2_GndOutIn -> cleaned footprints:SOT-223-3_TabPin2_GndOutIn
Changed lines of the file:
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@@
       (effects (font (size 1.27 1.27)))
     )
-    (property "Footprint" "Modified:SOT-223-3_TabPin2_GndOutIn" (at 91.44 26.67 0)
+    (property "Footprint" "cleaned footprints:SOT-223-3_TabPin2_GndOutIn" (at 91.44 26.67 0)
       (effects (font (size 1.27 1.27)) hide)
     )
